Commit message: Update anymal_c urdf joint position limits - https://github.com/google-deepmind/mujoco_menagerie/blob/main/anybotics_anymal_c/anymal_c.xml

File: assets/legged_gym/robots/anymal_c/urdf/anymal_c.urdf (robot description, URDF)
Before this commit: robot anymal, 77 links, 76 joints
Joints:
- joint LF_HAA: limit effort=80.0 velocity=20. -> lower=-0.72 upper=0.49 effort=80.0 velocity=20.
- joint LF_HFE: limit effort=80.0 velocity=20. -> lower=-9.42478 upper=9.42478 effort=80.0 velocity=20.
- joint LF_KFE: limit effort=80.0 velocity=20. -> lower=-9.42478 upper=9.42478 effort=80.0 velocity=20.
- joint LH_HAA: limit effort=80.0 velocity=20. -> lower=-0.72 upper=0.49 effort=80.0 velocity=20.
- joint LH_HFE: limit effort=80.0 velocity=20. -> lower=-9.42478 upper=9.42478 effort=80.0 velocity=20.
- joint LH_KFE: limit effort=80.0 velocity=20. -> lower=-9.42478 upper=9.42478 effort=80.0 velocity=20.
- joint RF_HAA: limit effort=80.0 velocity=20. -> lower=-0.49 upper=0.72 effort=80.0 velocity=20.
- joint RF_HFE: limit effort=80.0 velocity=20. -> lower=-9.42478 upper=9.42478 effort=80.0 velocity=20.
- joint RF_KFE: limit effort=80.0 velocity=20. -> lower=-9.42478 upper=9.42478 effort=80.0 velocity=20.
- joint RH_HAA: limit effort=80.0 velocity=20. -> lower=-0.49 upper=0.72 effort=80.0 velocity=20.
- joint RH_HFE: limit effort=80.0 velocity=20. -> lower=-9.42478 upper=9.42478 effort=80.0 velocity=20.
- joint RH_KFE: limit effort=80.0 velocity=20. -> lower=-9.42478 upper=9.42478 effort=80.0 velocity=20.
